Commit message: <sim> URDF: LiDAR/Camera 互换位置, LiDAR +76mm Camera -76mm + 去掉angle filter
- laser_z_world: 0.121→0.197, camera_z_world: 0.180→0.104
- sensors.launch.py: 去掉 laser_filter (雷达已放顶层360°无遮挡)
- 新增 laser_filter.yaml (保留备用, 后续如需裁剪可用)

File: app/src/robot_bringup/urdf/robot.xacro (robot description, xacro)
@@ -26,7 +26,7 @@
 	<!-- Sensor positions: absolute above ground (used for computing relative z) -->
 	<xacro:property name="laser_x"       value="0.1025"/>
-	<xacro:property name="laser_z_world" value="0.121"/>
+	<xacro:property name="laser_z_world" value="0.197"/>
 	<xacro:property name="camera_x"      value="0.1525"/>
-	<xacro:property name="camera_z_world" value="0.180"/>
+	<xacro:property name="camera_z_world" value="0.104"/>
 	<xacro:property name="imu_x"         value="0.0325"/>
 	<xacro:property name="imu_y"         value="0.0"/>

Commit message: <bringup> IMU标定: STM32陀螺零偏 0.6→<0.2°/s + WHEEL_BALANCE 0.003→0.001 + SLAM参数收紧 + URDF laser_frame→laser + fetch_app简化

File: app/src/robot_bringup/urdf/robot.xacro (robot description, xacro)
@@ -218,5 +218,5 @@
 	<xacro:lidar_pillar name="lidar_pillar_120" x="0.085"  y="0.0303"/>
 	<xacro:lidar_pillar name="lidar_pillar_240" x="0.085"  y="-0.0303"/>
-	<link name="laser_frame">
+	<link name="laser">
 		<visual>
 			<geometry><cylinder radius="0.035" length="0.02"/></geometry>
@@ -227,5 +227,5 @@
 	<joint name="laser_joint" type="fixed">
 		<parent link="base_link"/>
-		<child link="laser_frame"/>
+		<child link="laser"/>
 		<origin xyz="${laser_x} 0 ${laser_z}" rpy="0 0 0"/>
 	</joint>
